File: LaserDriverTest/LaserDriverTest.kicad_sch (KiCad schematic)
At the start: 10 parts, among them J1 Conn_01x02_Pin, J2 Conn_01x02_Pin, J3 Conn_01x07_Pin, J4 Conn_01x02_Pin

Commit message: Updated with product links
Parts:
- LT3083: value LT3083IT-PBF -> LT3083ET-PBF
Changed lines of the file:
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@@
 			)
 		)
-		(property "Value" "LT3083IT-PBF"
+		(property "Value" "LT3083ET-PBF"
 			(at 68.58 29.21 0)
 			(effects
@@
 			)
 		)
-		(property "Datasheet" "LT3083IT-40PBF"
+		(property "Datasheet" "LT3083ET-40PBF"
 			(at 35.56 36.83 0)
 			(effects
@@
 			)
 		)
-		(property "Description" ""
+		(property "Description" "https://mou.sr/4keM01S"
 			(at 35.56 36.83 0)
 			(effects
@@
 			)
 		)
-		(property "Datasheet" "AD5293BRUZ-100"
+		(property "Datasheet" "AD5293BRUZ-20"
 			(at 35.56 64.77 0)
 			(effects
@@
 			)
 		)
-		(property "Description" ""
+		(property "Description" "https://mou.sr/4dheQwe"
 			(at 35.56 64.77 0)
 			(effects
